File: MD-5.kicad_sch (KiCad schematic)
At the start: 4 parts

Commit message: harf bridge
Parts:
- added D? (x2): D, symbol Device:D
- added FB? (x2): FerriteBead_Small, symbol Device:FerriteBead_Small
- added Q? (x2): BSC025N08LS5, Package_TO_SOT_SMD_additional:infineon_PG-HSOG-8-1, symbol Transistor_FET_additional:BSC025N08LS5
- added R? (x2): R, symbol Device:R
Connections:
- net AHG: now also D?.1 (K), R?.1
- net AOUT: now also Q?.1 (S), Q?.2 (S), Q?.3 (S), Q?.5 (D), Q?.6 (D), Q?.7 (D), Q?.8 (D)
- net GND: now also Q?.1 (S), Q?.2 (S), Q?.3 (S)
- net LHG renamed ALG
- net ALG: now also D?.1 (K), R?.2
- new net: FB?.1, R?.2
- new net: D?.2 (A), FB?.2, Q?.4 (G) (x2)
- new net: FB?.1, R?.1
- new net VCC: Q?.5 (D), Q?.6 (D), Q?.7 (D), Q?.8 (D)

Commit message: on
Connections:
- net GND: now also U?.4 (GNDI); no longer C?.2, Q?.1 (S), Q?.2 (S), Q?.3 (S), U?.9 (GNDB)
- net AHIN: now reaches U?.1 (INA)
- net ALIN: now reaches U?.2 (INB)
- net +3V3: now reaches U?.3 (VDDI)
- net +3V3: now also U?.8 (SLDON)
- net DISABLE: now reaches U?.5 (DISABLE)
- new net GNDPWR: C?.2, Q?.1 (S), Q?.2 (S), Q?.3 (S), U?.9 (GNDB)
Changed lines of the file:
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@@
   (junction (at 162.56 58.42) (diameter 0) (color 0 0 0 0)
   )
+  (junction (at 120.65 58.42) (diameter 0) (color 0 0 0 0)
+  )
   (junction (at 175.26 50.8) (diameter 0) (color 0 0 0 0)
   )
@@
     (stroke (width 0) (type default) (color 0 0 0 0))
   )
+  (wire (pts (xy 121.92 60.96) (xy 129.54 60.96))
+    (stroke (width 0) (type default) (color 0 0 0 0))
+  )
   (wire (pts (xy 209.55 45.72) (xy 212.09 45.72))
     (stroke (width 0) (type default) (color 0 0 0 0))
@@
     (stroke (width 0) (type default) (color 0 0 0 0))
   )
+  (wire (pts (xy 120.65 58.42) (xy 120.65 68.58))
+    (stroke (width 0) (type default) (color 0 0 0 0))
+  )
   (wire (pts (xy 162.56 76.2) (xy 162.56 73.66))
     (stroke (width 0) (type default) (color 0 0 0 0))
@@
     (stroke (width 0) (type default) (color 0 0 0 0))
   )
+  (wire (pts (xy 121.92 63.5) (xy 129.54 63.5))
+    (stroke (width 0) (type default) (color 0 0 0 0))
+  )
   (wire (pts (xy 196.85 63.5) (xy 194.31 66.04))
     (stroke (width 0) (type default) (color 0 0 0 0))
@@
     (stroke (width 0) (type default) (color 0 0 0 0))
   )
+  (wire (pts (xy 123.19 55.88) (xy 129.54 55.88))
+    (stroke (width 0) (type default) (color 0 0 0 0))
+  )
   (wire (pts (xy 214.63 68.58) (xy 220.98 68.58))
     (stroke (width 0) (type default) (color 0 0 0 0))
@@
     (stroke (width 0) (type default) (color 0 0 0 0))
   )
+  (wire (pts (xy 121.92 60.96) (xy 118.11 64.77))
+    (stroke (width 0) (type default) (color 0 0 0 0))
+  )
   (wire (pts (xy 212.09 45.72) (xy 214.63 48.26))
     (stroke (width 0) (type default) (color 0 0 0 0))
   )
+  (wire (pts (xy 120.65 48.26) (xy 120.65 58.42))
+    (stroke (width 0) (type default) (color 0 0 0 0))
+  )
   (wire (pts (xy 175.26 48.26) (xy 175.26 50.8))
     (stroke (width 0) (type default) (color 0 0 0 0))
@@
     (stroke (width 0) (type default) (color 0 0 0 0))
   )
+  (wire (pts (xy 123.19 53.34) (xy 129.54 53.34))
+    (stroke (width 0) (type default) (color 0 0 0 0))
+  )
   (wire (pts (xy 201.93 63.5) (xy 196.85 63.5))
     (stroke (width 0) (type default) (color 0 0 0 0))
@@
     (stroke (width 0) (type default) (color 0 0 0 0))
   )
+  (wire (pts (xy 118.11 64.77) (xy 118.11 76.2))
+    (stroke (width 0) (type default) (color 0 0 0 0))
+  )
   (wire (pts (xy 201.93 45.72) (xy 196.85 45.72))
     (stroke (width 0) (type default) (color 0 0 0 0))
@@
     (stroke (width 0) (type default) (color 0 0 0 0))
   )
+  (wire (pts (xy 123.19 71.12) (xy 129.54 71.12))
+    (stroke (width 0) (type default) (color 0 0 0 0))
+  )
   (wire (pts (xy 214.63 68.58) (xy 214.63 71.12))
     (stroke (width 0) (type default) (color 0 0 0 0))
   )
+  (wire (pts (xy 123.19 71.12) (xy 120.65 68.58))
+    (stroke (width 0) (type default) (color 0 0 0 0))
+  )
   (wire (pts (xy 194.31 48.26) (xy 194.31 55.88))
+    (stroke (width 0) (type default) (color 0 0 0 0))
+  )
+  (wire (pts (xy 120.65 58.42) (xy 129.54 58.42))
     (stroke (width 0) (type default) (color 0 0 0 0))
   )
@@
     (effects (font (size 1.27 1.27)) (justify right bottom))
   )
+  (label "AHIN" (at 123.19 53.34 0)
+    (effects (font (size 1.27 1.27)) (justify left bottom))
+  )
   (label "AOUT" (at 168.91 58.42 180)
     (effects (font (size 1.27 1.27)) (justify right bottom))
+  )
+  (label "ALIN" (at 123.19 55.88 0)
+    (effects (font (size 1.27 1.27)) (justify left bottom))
+  )
+  (label "DISABLE" (at 121.92 63.5 0)
+    (effects (font (size 1.27 1.27)) (justify left bottom))
   )
   (label "AOUT" (at 238.76 62.23 180)
@@
     (pin "2")
   )
-  (symbol (lib_id "power:GND") (at 162.56 76.2 0) (unit 1)
-    (in_bom yes) (on_board yes)
-    (property "Reference" "#PWR?" (id 0) (at 162.56 82.55 0)
-      (effects (font (size 1.27 1.27)) hide)
-    )
-    (property "Value" "GND" (id 1) (at 162.687 80.5942 0))
-    (property "Footprint" "" (id 2) (at 162.56 76.2 0)
-      (effects (font (size 1.27 1.27)) hide)
-    )
-    (property "Datasheet" "" (id 3) (at 162.56 76.2 0)
-      (effects (font (size 1.27 1.27)) hide)
-    )
-    (pin "1")
-  )
   (symbol (lib_id "power:+12V") (at 175.26 48.26 0) (unit 1)
     (in_bom yes) (on_board yes)
@@
     (pin "1")
   )
+  (symbol (lib_id "power:GNDPWR") (at 228.6 76.2 0) (unit 1)
+    (in_bom yes) (on_board yes) (fields_autoplaced)
+    (property "Reference" "#PWR?" (id 0) (at 228.6 81.28 0)
+      (effects (font (size 1.27 1.27)) hide)
+    )
+    (property "Value" "GNDPWR" (id 1) (at 228.473 80.3561 0))
+    (property "Footprint" "" (id 2) (at 228.6 77.47 0)
+      (effects (font (size 1.27 1.27)) hide)
+    )
+    (property "Datasheet" "" (id 3) (at 228.6 77.47 0)
+      (effects (font (size 1.27 1.27)) hide)
+    )
+    (pin "1")
+  )
+  (symbol (lib_id "power:+3.3V") (at 120.65 48.26 0) (unit 1)
+    (in_bom yes) (on_board yes) (fields_autoplaced)
+    (property "Reference" "#PWR?" (id 0) (at 120.65 52.07 0)
+      (effects (font (size 1.27 1.27)) hide)
+    )
+    (property "Value" "+3.3V" (id 1) (at 120.65 44.6555 0))
+    (property "Footprint" "" (id 2) (at 120.65 48.26 0)
+      (effects (font (size 1.27 1.27)) hide)
+    )
+    (property "Datasheet" "" (id 3) (at 120.65 48.26 0)
+      (effects (font (size 1.27 1.27)) hide)
+    )
+    (pin "1")
+  )
   (symbol (lib_id "Device:FerriteBead_Small") (at 209.55 55.88 90) (unit 1)
     (in_bom yes) (on_board yes) (fields_autoplaced)
@@
     (pin "2")
   )
+  (symbol (lib_id "power:GND") (at 118.11 76.2 0) (unit 1)
+    (in_bom yes) (on_board yes) (fields_autoplaced)
+    (property "Reference" "#PWR?" (id 0) (at 118.11 82.55 0)
+      (effects (font (size 1.27 1.27)) hide)
+    )
+    (property "Value" "GND" (id 1) (at 118.11 80.7625 0))
+    (property "Footprint" "" (id 2) (at 118.11 76.2 0)
+      (effects (font (size 1.27 1.27)) hide)
+    )
+    (property "Datasheet" "" (id 3) (at 118.11 76.2 0)
+      (effects (font (size 1.27 1.27)) hide)
+    )
+    (pin "1")
+  )
   (symbol (lib_id "Device:FerriteBead_Small") (at 209.55 73.66 90) (unit 1)
     (in_bom yes) (on_board yes) (fields_autoplaced)
@@
     (pin "1")
     (pin "2")
-  )
-  (symbol (lib_id "power:GND") (at 228.6 76.2 0) (unit 1)
-    (in_bom yes) (on_board yes)
-    (property "Reference" "#PWR?" (id 0) (at 228.6 82.55 0)
-      (effects (font (size 1.27 1.27)) hide)
-    )
-    (property "Value" "GND" (id 1) (at 228.727 80.5942 0))
-    (property "Footprint" "" (id 2) (at 228.6 76.2 0)
-      (effects (font (size 1.27 1.27)) hide)
-    )
-    (property "Datasheet" "" (id 3) (at 228.6 76.2 0)
-      (effects (font (size 1.27 1.27)) hide)
-    )
-    (pin "1")
   )
   (symbol (lib_id "power:VCC") (at 228.6 48.26 0) (unit 1)
@@
     (pin "8")
   )
+  (symbol (lib_id "power:GNDPWR") (at 162.56 76.2 0) (unit 1)
+    (in_bom yes) (on_board yes) (fields_autoplaced)
+    (property "Reference" "#PWR?" (id 0) (at 162.56 81.28 0)
+      (effects (font (size 1.27 1.27)) hide)
+    )
+    (property "Value" "GNDPWR" (id 1) (at 162.433 80.3561 0))
+    (property "Footprint" "" (id 2) (at 162.56 77.47 0)
+      (effects (font (size 1.27 1.27)) hide)
+    )
+    (property "Datasheet" "" (id 3) (at 162.56 77.47 0)
+      (effects (font (size 1.27 1.27)) hide)
+    )
+    (pin "1")
+  )
   (sheet_instances
     (path "/" (page "1"))
   )
   (symbol_instances
-    (path "/00000000-0000-0000-0000-000061c7fa86"
-      (reference "#PWR?") (unit 1) (value "GND") (footprint "")
-    )
     (path "/00000000-0000-0000-0000-000061c8075c"
       (reference "#PWR?") (unit 1) (value "+12V") (footprint "")
     )
-    (path "/7a8c1bb7-139d-47ec-b102-888dd8d68843"
+    (path "/01b6cbe6-9563-4aab-bfd8-ea939ff3d79a"
+      (reference "#PWR?") (unit 1) (value "GNDPWR") (footprint "")
+    )
+    (path "/0577c14e-2a48-4266-b611-ad9a9e537b1a"
+      (reference "#PWR?") (unit 1) (value "+3.3V") (footprint "")
+    )
+    (path "/61a355d9-5231-4699-9738-3ec704d44035"
       (reference "#PWR?") (unit 1) (value "GND") (footprint "")
     )
@@
       (reference "#PWR?") (unit 1) (value "VCC") (footprint "")
     )
+    (path "/fe45c4a1-51cd-4239-8a94-676cbced478b"
+      (reference "#PWR?") (unit 1) (value "GNDPWR") (footprint "")
+    )
     (path "/00000000-0000-0000-0000-000061c799c6"

Commit message: maikontuika
Parts:
- added C? (x2): 10uF, Capacitor_SMD:C_0805_2012Metric, symbol Device:C
- added C? (x2): 10uF, Capacitor_SMD:C_1206_3216Metric, symbol Device:C
- added D? (x7): D, symbol Device:D
- added FB? (x2): FerriteBead_Small, Inductor_SMD:L_0603_1608Metric, symbol Device:FerriteBead_Small
- added Q? (x2): BSC025N08LS5, Package_TO_SOT_SMD_additional:infineon_PG-HSOG-8-1, symbol Transistor_FET_additional:BSC025N08LS5
- added R? (x2): 7.5R, Resistor_SMD:R_0603_1608Metric, symbol Device:R
- added R? (x4): 5R, Resistor_SMD:R_0603_1608Metric, symbol Device:R
- added U?: STM32F303K8Tx, Package_QFP:LQFP-32_7x7mm_P0.8mm, symbol MCU_ST_STM32F3:STM32F303K8Tx
- added U?: MCP2551-I-SN, Package_SO:SOIC-8_3.9x4.9mm_P1.27mm, symbol Interface_CAN_LIN:MCP2551-I-SN
- added U?: 2EDF7175, Package_SO:SOIC-16_3.9x9.9mm_P1.27mm, symbol Driver_FET_additional:2EDF7175
- C? (x2): value C -> 10uF; footprint (none) -> Capacitor_SMD:C_0805_2012Metric
- FB? (x2): footprint (none) -> Inductor_SMD:L_0603_1608Metric
- R? (x2): value R -> 7.5R; footprint (none) -> Resistor_SMD:R_0603_1608Metric
Connections:
- net +12V: now also C?.1, D?.2 (A), U?.11 (VDDB)
- net +3V3: now also U?.1 (VDD), U?.17 (VDD), U?.3 (VDDI), U?.5 (VDDA), U?.8 (SLDON)
- net AHG: now also R?.2; no longer D?.1 (K)
- net AHIN: now also U?.18 (PA8)
- net ALG: now also R?.2; no longer D?.1 (K)
- net ALIN: now also U?.13 (PA7)
- net AOUT: now also D?.1 (K), D?.2 (A)
- net DISABLE: now also U?.28 (PB5), U?.5 (DISABLE)
- net GND: now also U?.16 (VSS), U?.2 (VSS), U?.32 (VSS), U?.4 (GNDI)
- net GNDPWR: now also C?.2, C?.2, C?.2, D?.2 (A), D?.2 (A), Q?.1 (S), Q?.2 (S), Q?.3 (S), U?.9 (GNDB)
- net VCC: now also C?.1, C?.1, D?.1 (K), D?.1 (K), Q?.5 (D), Q?.6 (D), Q?.7 (D), Q?.8 (D)
- new net: C?.1, D?.1 (K), U?.16 (VDDA)
- new net: FB?.1, R?.1
- new net: D?.1 (K), R?.1 (x4)
- new net: FB?.1, R?.2
- new net: D?.2 (A), FB?.2, Q?.4 (G) (x2)
- new net +5V: U?.3 (VDD)
- new net BHG: R?.1, R?.2, U?.15 (OUTA)
- new net BHIN: U?.1 (INA), U?.19 (PA9)
- new net BLG: R?.2, R?.2, U?.10 (OUTB)
- new net BLIN: U?.14 (PB0), U?.2 (INB)
- new net BOOT0: U?.31 (BOOT0)
- new net BOUT: C?.2, D?.1 (K), D?.2 (A), Q?.1 (S), Q?.2 (S), Q?.3 (S), Q?.5 (D), Q?.6 (D), Q?.7 (D), Q?.8 (D), U?.14 (GNDA)
- new net CAN_RX: U?.21 (PA11), U?.4 (RXD)
- new net CAN_TX: U?.1 (TXD), U?.22 (PA12)
- new net NRST: U?.4 (NRST)
- new net OSC_IN: U?.2 (PF0)
- new net OSC_OUT: U?.3 (PF1)
- new net PWM_IN1: U?.11 (PA5)
- new net PWM_IN2: U?.12 (PA6)
- new net SWCLK: U?.24 (PA14)
- new net SWDIO: U?.23 (PA13)
Other:
- moved on the sheet: D?

Commit message: CANHL
Parts:
- added R?: 120R, Resistor_SMD:R_0603_1608Metric, symbol Device:R
Connections:
- net CANL: now reaches U?.6 (CANL)
- net CANL: now also R?.2
- net CANH: now reaches U?.7 (CANH)
- net CANH: now also R?.1
Changed lines of the file:
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@@
   (junction (at 194.31 124.46) (diameter 0) (color 0 0 0 0)
   )
+  (junction (at 92.71 168.91) (diameter 0) (color 0 0 0 0)
+  )
   (junction (at 120.65 109.22) (diameter 0) (color 0 0 0 0)
   )
@@
   (junction (at 214.63 55.88) (diameter 0) (color 0 0 0 0)
   )
+  (junction (at 92.71 161.29) (diameter 0) (color 0 0 0 0)
+  )
   (junction (at 162.56 73.66) (diameter 0) (color 0 0 0 0)
   )
@@
     (stroke (width 0) (type default) (color 0 0 0 0))
   )
+  (wire (pts (xy 86.36 162.56) (xy 87.63 161.29))
+    (stroke (width 0) (type default) (color 0 0 0 0))
+  )
   (wire (pts (xy 123.19 104.14) (xy 129.54 104.14))
     (stroke (width 0) (type default) (color 0 0 0 0))
@@
     (stroke (width 0) (type default) (color 0 0 0 0))
   )
+  (wire (pts (xy 81.28 167.64) (xy 86.36 167.64))
+    (stroke (width 0) (type default) (color 0 0 0 0))
+  )
   (wire (pts (xy 154.94 53.34) (xy 157.48 50.8))
     (stroke (width 0) (type default) (color 0 0 0 0))
@@
     (stroke (width 0) (type default) (color 0 0 0 0))
   )
+  (wire (pts (xy 86.36 167.64) (xy 87.63 168.91))
+    (stroke (width 0) (type default) (color 0 0 0 0))
+  )
   (wire (pts (xy 123.19 55.88) (xy 129.54 55.88))
     (stroke (width 0) (type default) (color 0 0 0 0))
@@
     (stroke (width 0) (type default) (color 0 0 0 0))
   )
+  (wire (pts (xy 92.71 161.29) (xy 104.14 161.29))
+    (stroke (width 0) (type default) (color 0 0 0 0))
+  )
   (wire (pts (xy 66.04 132.08) (xy 66.04 129.54))
     (stroke (width 0) (type default) (color 0 0 0 0))
@@
     (stroke (width 0) (type default) (color 0 0 0 0))
   )
+  (wire (pts (xy 92.71 168.91) (xy 104.14 168.91))
+    (stroke (width 0) (type default) (color 0 0 0 0))
+  )
   (wire (pts (xy 172.72 101.6) (xy 175.26 101.6))
     (stroke (width 0) (type default) (color 0 0 0 0))
@@
     (stroke (width 0) (type default) (color 0 0 0 0))
   )
+  (wire (pts (xy 87.63 161.29) (xy 92.71 161.29))
+    (stroke (width 0) (type default) (color 0 0 0 0))
+  )
   (wire (pts (xy 162.56 63.5) (xy 162.56 66.04))
     (stroke (width 0) (type default) (color 0 0 0 0))
@@
   )
   (wire (pts (xy 194.31 48.26) (xy 194.31 55.88))
+    (stroke (width 0) (type default) (color 0 0 0 0))
+  )
+  (wire (pts (xy 87.63 168.91) (xy 92.71 168.91))
+    (stroke (width 0) (type default) (color 0 0 0 0))
+  )
+  (wire (pts (xy 81.28 162.56) (xy 86.36 162.56))
     (stroke (width 0) (type default) (color 0 0 0 0))
   )
@@
     (effects (font (size 1.27 1.27)) (justify left bottom))
   )
+  (label "CANL" (at 104.14 168.91 180)
+    (effects (font (size 1.27 1.27)) (justify right bottom))
+  )
   (label "DISABLE" (at 121.92 63.5 0)
     (effects (font (size 1.27 1.27)) (justify left bottom))
@@
   (label "BLIN" (at 123.19 106.68 0)
     (effects (font (size 1.27 1.27)) (justify left bottom))
+  )
+  (label "CANH" (at 104.14 161.29 180)
+    (effects (font (size 1.27 1.27)) (justify right bottom))
   )
   (label "BHIN" (at 85.09 109.22 180)
@@
     )
     (pin "1")
+  )
+  (symbol (lib_id "Device:R") (at 92.71 165.1 0) (unit 1)
+    (in_bom yes) (on_board yes) (fields_autoplaced)
+    (property "Reference" "R?" (id 0) (at 94.488 164.1915 0)
+      (effects (font (size 1.27 1.27)) (justify left))
+    )
+    (property "Value" "120R" (id 1) (at 94.488 166.9666 0)
+      (effects (font (size 1.27 1.27)) (justify left))
+    )
+    (property "Footprint" "Resistor_SMD:R_0603_1608Metric" (id 2) (at 90.932 165.1 90)
+      (effects (font (size 1.27 1.27)) hide)
+    )
+    (property "Datasheet" "~" (id 3) (at 92.71 165.1 0)
+      (effects (font (size 1.27 1.27)) hide)
+    )
+    (pin "1")
+    (pin "2")
   )
   (symbol (lib_id "Device:D") (at 248.92 68.58 270) (unit 1)
@@
       (reference "R?") (unit 1) (value "7.5R") (footprint "Resistor_SMD:R_0603_1608Metric")
     )
+    (path "/254965a0-962f-4583-bec6-6de0a1529408"
+      (reference "R?") (unit 1) (value "120R") (footprint "Resistor_SMD:R_0603_1608Metric")
+    )
     (path "/2e10d874-a310-4b7f-8ae4-4d1bfee0cc73"

Commit message: mcushuuhen
Parts:
- added C? (x2): C, Capacitor_SMD:C_0603_1608Metric, symbol Device:C
- added C?: 0.1uF, Capacitor_SMD:C_0603_1608Metric, symbol Device:C
- added R?: 10kR, Resistor_SMD:R_0603_1608Metric, symbol Device:R
- added SW?: SW_Push, Button_Switch_additional:TVAF06-A020B-R, symbol Switch:SW_Push
- added Y?: Crystal_GND24, Crystal:Crystal_SMD_3225-4Pin_3.2x2.5mm, symbol Device:Crystal_GND24
Connections:
- net BOOT0: now also R?.2
- net GND: now also C?.2, C?.2, C?.2, R?.1, SW?.1, Y?.2, Y?.4
- net NRST: now also C?.1, SW?.2
- net OSC_IN: now also C?.1, Y?.3
- net OSC_OUT: now also C?.1, Y?.1
Other:
- moved on the sheet: C?, D?, FB?, Q?, R?, U?

Commit message: sche fin?
Parts:
- added C? (x3): 10uF, Capacitor_SMD:C_0805_2012Metric, symbol Device:C
- added C?: 10uF, Capacitor_SMD:C_1206_3216Metric, symbol Device:C
- added J?: Conn_02x24_Odd_Even, Connector_PinHeader_2.54mm:PinHeader_2x24_P2.54mm_Horizontal, symbol Connector_Generic:Conn_02x24_Odd_Even
- added J?: Conn_02x07_Odd_Even, Connector_PinHeader_1.27mm:PinHeader_2x07_P1.27mm_Vertical_SMD, symbol Connector_Generic:Conn_02x07_Odd_Even
- added R?: 10kR, Resistor_SMD:R_0603_1608Metric, symbol Device:R
- added U?: L7812, Package_TO_SOT_SMD:TO-252-2, symbol Regulator_Linear:L7812
- added U?: MCP1792-3302H, Package_TO_SOT_SMD:SOT-23, symbol Regulator_Linear:MCP1700-3302E_SOT23
- C? (x2): value C -> 22pF
Connections:
- net +12V: now also C?.1, U?.3 (OUT)
- net +3V3: now also C?.1, J?.3 (Pin_3), J?.48 (Pin_48), U?.2 (VO)
- net +5V: now also C?.1, J?.47 (Pin_47), U?.3 (VI)
- net CANH: now also J?.45 (Pin_45)
- net CANL: now also J?.43 (Pin_43)
- net GND: now also C?.2, C?.2, J?.11 (Pin_11), J?.41 (Pin_41), J?.42 (Pin_42), J?.5 (Pin_5), J?.7 (Pin_7), R?.1, U?.1 (GND)
- net GNDPWR: now also C?.2, C?.2, J?.1 (Pin_1), J?.10 (Pin_10), J?.11 (Pin_11), J?.12 (Pin_12), J?.13 (Pin_13), J?.14 (Pin_14), J?.15 (Pin_15), J?.16 (Pin_16), J?.17 (Pin_17), J?.18 (Pin_18), J?.19 (Pin_19), J?.2 (Pin_2), J?.20 (Pin_20), J?.3 (Pin_3), J?.4 (Pin_4), J?.5 (Pin_5), J?.6 (Pin_6), J?.7 (Pin_7), J?.8 (Pin_8), J?.9 (Pin_9), U?.2 (GND)
- net NRST: now also J?.12 (Pin_12)
- net PWM_IN1: now also J?.46 (Pin_46)
- net PWM_IN2: now also J?.44 (Pin_44)
- net SWCLK: now also J?.6 (Pin_6)
- net SWDIO: now also J?.4 (Pin_4)
- net VCC: now also C?.1, J?.21 (Pin_21), J?.22 (Pin_22), J?.23 (Pin_23), J?.24 (Pin_24), J?.25 (Pin_25), J?.26 (Pin_26), J?.27 (Pin_27), J?.28 (Pin_28), J?.29 (Pin_29), J?.30 (Pin_30), J?.31 (Pin_31), J?.32 (Pin_32), J?.33 (Pin_33), J?.34 (Pin_34), J?.35 (Pin_35), J?.36 (Pin_36), J?.37 (Pin_37), J?.38 (Pin_38), J?.39 (Pin_39), J?.40 (Pin_40), U?.1 (IN)
- net VCP_TX: now reaches U?.29 (PB6)
- net VCP_TX: now also J?.14 (Pin_14)
- net VCP_RX: now reaches U?.30 (PB7)
- net VCP_RX: now also J?.13 (Pin_13)
- net at U?.8 (Rs): now also R?.2
Other:
- moved on the sheet: C?, D?, FB?, Q?, R?, U?

Commit message: うわーー
Parts:
- added C16, C17: 33uF, Capacitor_SMD:CP_Elec_6.3x7.7, symbol Device:C_Polarized
- added C20, C3, C6, C7, C8: 0.1uF, Capacitor_SMD:C_0603_1608Metric, symbol Device:C
- added D1, D2: WS2812C, LED_additional:LED_2020Metric_WS2812C_2.0x2.0mm_P1.0mm, symbol LED_additional:WS2812C
- added D3: LED, LED_SMD:LED_0603_1608Metric, symbol Device:LED
- added D?: D_TVS, symbol Device:D_TVS
- added J3: Output, Connector_T_connector:T_connecter_female_horizontal, symbol Connector:Conn_01x02_Female
- added R4: 10kR, Resistor_SMD:R_0603_1608Metric, symbol Device:R
- D10, D11, D12, D13: renamed from D?; value D -> CUHS20S60H3F; footprint (none) -> Diode_additional:D_US2A
- D4, D5, D6, D7, D8, D9: renamed from D?; value D -> 1N4148W; footprint (none) -> Diode_SMD:D_SOD-123
- FB1, FB2, FB3, FB4: renamed from FB?; value FerriteBead_Small -> 60Ohm 100MHz
- J2: renamed from J?; value Conn_02x24_Odd_Even -> Header_hol_02x24
- Q1, Q2, Q3, Q4: renamed from Q?; footprint Package_TO_SOT_SMD_additional:infineon_PG-HSOG-8-1 -> Package_TO_SOT_SMD:TDSON-8-1
- Y1: renamed from Y?; value Crystal_GND24 -> 16MHz
- gave numbers to parts that had none: 32
Connections:
- net +3V3: now also C6.1, C7.1, C8.1, R4.2
- net +5V: now also C20.1, C3.1, D1.4 (VDD), D2.4 (VDD)
- net AOUT: now also J3.1 (Pin_1)
- net BOUT: now also J3.2 (Pin_2)
- net DISABLE: now also D3.1 (K)
- net GND: now also C20.2, C3.2, C6.2, C7.2, C8.2, D1.2 (VSS), D2.2 (VSS)
- net GNDPWR: now also C16.2, C17.2, D?.2 (A2)
- net VCC: now also C16.1, C17.1, D?.1 (A1)
- net NeoPixel: now reaches U2.15 (PB1)
- net NeoPixel: now also D1.3 (DIN)
- new net: D3.2 (A), R4.1
- new net: D1.1 (DOUT), D2.3 (DIN)
Other:
- moved on the sheet: C18, C19, C5, C9, J2, R1, R3, U1, U3
