File: MD-5.kicad_pcb (KiCad board)
At the start: 2 copper layers, 61 x 40 mm, 65 parts, among them J1 Conn_02x07_Odd_Even, J2 Header_hol_02x24, J3 Output, Q1 BSC025N08LS5, Q2 BSC025N08LS5, Q3 BSC025N08LS5, Q4 BSC025N08LS5, SW1 SW_Push, U1 MCP2551-I-SN, U2 STM32F303K8Tx, U3 MCP1792-3302H, U4 2EDF7175, U5 2EDF7175, U6 L7812, Y1 16MHz

Commit message: comp
Routing:
- net /ALG: track 1.90 -> 38.2 mm, vias 0 -> 2
- net /BLG: track 1.90 -> 37.5 mm, vias 0 -> 2
- net GNDPWR: track 0.00 -> 25.8 mm, vias 0 -> 2
- net GND: track 17.3 -> 0.00 mm, vias 62 -> 69
- net /BOUT: track 2.48 -> 17.3 mm, vias 0 -> 66
- net /AOUT: track 2.48 -> 17.3 mm, vias 0 -> 69
- net /DISABLE: track 18.3 -> 30.3 mm, vias 2 -> 3
- net /NeoPixel: track 29.6 -> 24.9 mm, vias 4 -> 2
- net +5V: track 58.9 -> 54.4 mm
- net /NRST: track 35.9 -> 32.7 mm
- net /VCP_RX: track 25.8 -> 23.6 mm
- net /VCP_TX: track 27.3 -> 25.2 mm
- net /CAN_RX: track 29.9 -> 31.6 mm
- net +3V3: track 90.3 -> 88.8 mm, vias 7 -> 11
- net /CAN_TX: track 24.9 -> 26.0 mm
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- added copper zone on B.Cu, net /AOUT
- added copper zone on F.Cu, net /AOUT
- added copper zone on B.Cu, net /BOUT
- added copper zone on F.Cu, net /BOUT
- added copper zone on F.Cu, net GNDPWR
- added copper zone on B.Cu, net VCC
