File: MD-5.kicad_pcb (KiCad board)
At the start: 2 copper layers, 61 x 40 mm, 65 parts, among them J1 Conn_02x07_Odd_Even, J2 Header_hol_02x24, J3 Output, Q1 BSC025N08LS5, Q2 BSC025N08LS5, Q3 BSC025N08LS5, Q4 BSC025N08LS5, SW1 SW_Push, U1 MCP2551-I-SN, U2 STM32F303K8Tx, U3 MCP1792-3302H, U4 2EDF7175, U5 2EDF7175, U6 L7812, Y1 16MHz

Commit message: silk
Other:
- board text added: "Designed by paripal"
- board text added: "MD-5_v0"
Changed lines of the file:
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@@
   (gr_line (start 190.5 100.33) (end 132.08 100.33) (layer "Edge.Cuts") (width 0.1))
   (gr_arc (start 130.81 101.6) (mid 131.181974 100.701974) (end 132.08 100.33) (layer "Edge.Cuts") (width 0.1))
+  (gr_text "MD-5_v0" (at 135.509 122.047 270) (layer "B.SilkS")
+    (effects (font (size 1.5 1.5) (thickness 0.2)) (justify mirror))
+  )
+  (gr_text "Designed by paripal" (at 133.35 119.507 270) (layer "B.SilkS")
+    (effects (font (size 1 1) (thickness 0.15)) (justify mirror))
+  )
   (segment (start 136.964489 102.609712) (end 137.339201 102.235) (width 0.25) (layer "F.Cu") (net 1))
   (segment (start 136.964489 104.560237) (end 136.964489 102.609712) (width 0.25) (layer "F.Cu") (net 1))
